File: easter.kicad_sch (KiCad schematic)
At the start: 27 parts, among them Q1 BC547, Q2 BC547, SW1 SW_Push_SPDT, SW2 Shake, SW3 SW_Push_SPDT

Commit message: Add solar test points
Parts:
- added TP1, TP2: TestPoint, TestPoint:TestPoint_THTPad_D2.0mm_Drill1.0mm, symbol Connector:TestPoint
Connections:
- net VDC: now also TP1.1
- net at D1.1 (K), Q1.3 (E), SC1.2 (-): now also TP2.1
Changed lines of the file:
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@@
   (junction (at 154.94 88.9) (diameter 0) (color 0 0 0 0)
   )
+  (junction (at 48.26 58.42) (diameter 0) (color 0 0 0 0)
+  )
   (junction (at 54.61 104.14) (diameter 0) (color 0 0 0 0)
   )
@@
   )
   (junction (at 179.07 88.9) (diameter 0) (color 0 0 0 0)
+  )
+  (junction (at 48.26 81.28) (diameter 0) (color 0 0 0 0)
   )
   (junction (at 83.82 88.9) (diameter 0) (color 0 0 0 0)
@@
     (stroke (width 0) (type default) (color 0 0 0 0))
   )
+  (wire (pts (xy 48.26 73.66) (xy 48.26 81.28))
+    (stroke (width 0) (type default) (color 0 0 0 0))
+  )
   (wire (pts (xy 109.22 78.74) (xy 109.22 77.47))
     (stroke (width 0) (type default) (color 0 0 0 0))
@@
     (stroke (width 0) (type default) (color 0 0 0 0))
   )
+  (wire (pts (xy 48.26 58.42) (xy 48.26 66.04))
+    (stroke (width 0) (type default) (color 0 0 0 0))
+  )
   (wire (pts (xy 154.94 86.36) (xy 154.94 88.9))
     (stroke (width 0) (type default) (color 0 0 0 0))
@@
     (stroke (width 0) (type default) (color 0 0 0 0))
   )
-  (wire (pts (xy 48.26 73.66) (xy 48.26 95.25))
-    (stroke (width 0) (type default) (color 0 0 0 0))
-  )
   (wire (pts (xy 54.61 104.14) (xy 67.31 104.14))
     (stroke (width 0) (type default) (color 0 0 0 0))
@@
     (stroke (width 0) (type default) (color 0 0 0 0))
   )
-  (wire (pts (xy 48.26 53.34) (xy 48.26 66.04))
+  (wire (pts (xy 48.26 53.34) (xy 48.26 58.42))
     (stroke (width 0) (type default) (color 0 0 0 0))
   )
@@
     (stroke (width 0) (type default) (color 0 0 0 0))
   )
+  (wire (pts (xy 48.26 81.28) (xy 48.26 95.25))
+    (stroke (width 0) (type default) (color 0 0 0 0))
+  )
   (wire (pts (xy 106.68 67.31) (xy 106.68 66.04))
     (stroke (width 0) (type default) (color 0 0 0 0))
@@
   (wire (pts (xy 154.94 78.74) (xy 154.94 71.12))
     (stroke (width 0) (type default) (color 0 0 0 0))
+  )
+  (symbol (lib_id "Connector:TestPoint") (at 48.26 81.28 90) (unit 1)
+    (in_bom yes) (on_board yes) (fields_autoplaced)
+    (property "Reference" "TP2" (id 0) (at 44.958 74.93 90))
+    (property "Value" "TestPoint" (id 1) (at 44.958 77.47 90))
+    (property "Footprint" "TestPoint:TestPoint_THTPad_D2.0mm_Drill1.0mm" (id 2) (at 48.26 76.2 0)
+      (effects (font (size 1.27 1.27)) hide)
+    )
+    (property "Datasheet" "~" (id 3) (at 48.26 76.2 0)
+      (effects (font (size 1.27 1.27)) hide)
+    )
+    (pin "1")
   )
   (symbol (lib_id "power:GND") (at 48.26 127 0) (unit 1)
@@
     (pin "1")
     (pin "2")
+  )
+  (symbol (lib_id "Connector:TestPoint") (at 48.26 58.42 90) (unit 1)
+    (in_bom yes) (on_board yes) (fields_autoplaced)
+    (property "Reference" "TP1" (id 0) (at 44.958 52.07 90))
+    (property "Value" "TestPoint" (id 1) (at 44.958 54.61 90))
+    (property "Footprint" "TestPoint:TestPoint_THTPad_D2.0mm_Drill1.0mm" (id 2) (at 48.26 53.34 0)
+      (effects (font (size 1.27 1.27)) hide)
+    )
+    (property "Datasheet" "~" (id 3) (at 48.26 53.34 0)
+      (effects (font (size 1.27 1.27)) hide)
+    )
+    (pin "1")
   )
   (symbol (lib_id "Device:R") (at 60.96 83.82 0) (unit 1)
@@
       (reference "SW3") (unit 1) (value "SW_Push_SPDT") (footprint "Button_Switch_THT:SW_Slide_1P2T_CK_OS102011MS2Q")
     )
-  )
+    (path "/16ca0079-b119-4057-8736-31120738f708"
+      (reference "TP1") (unit 1) (value "TestPoint") (footprint "TestPoint:TestPoint_THTPad_D2.0mm_Drill1.0mm")
+    )
+    (path "/0461edd4-b7ea-4d80-a7dc-ab1b81a9b8ff"
+      (reference "TP2") (unit 1) (value "TestPoint") (footprint "TestPoint:TestPoint_THTPad_D2.0mm_Drill1.0mm")
+    )
+  )
