File: hardware/easter.kicad_pcb (KiCad board)
At the start: 2 copper layers, 69.7 x 90.8 mm, 29 parts, among them Q1 BC547, Q2 BC547, SW1 SW_Push_SPDT, SW2 Shake, SW3 SW_Push_SPDT

Commit message: Updated links to libraries
Parts:
- BT1, BT2: footprint custom footprints:MP001179 -> CustomLocalLib:MP001179
- SC1: footprint custom footprints:KXOB25-03X4F-TR -> CustomLocalLib:KXOB25-03X4F-TR
