File: hardware/easter.kicad_sch (KiCad schematic)
At the start: 29 parts, among them Q1 BC547, Q2 BC547, SW1 SW_Push_SPDT, SW2 Shake, SW3 SW_Push_SPDT

Commit message: Updated links to libraries
Parts:
- BT1, BT2: footprint custom footprints:MP001179 -> CustomLocalLib:MP001179
- SC1: footprint custom footprints:KXOB25-03X4F-TR -> CustomLocalLib:KXOB25-03X4F-TR
Changed lines of the file:
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@@
 			)
 		)
-		(property "Footprint" "custom footprints:MP001179"
+		(property "Footprint" "CustomLocalLib:MP001179"
 			(at 215.9 79.756 90)
 			(effects
@@
 			)
 		)
-		(property "Footprint" "custom footprints:KXOB25-03X4F-TR"
+		(property "Footprint" "CustomLocalLib:KXOB25-03X4F-TR"
 			(at 48.26 69.596 90)
 			(effects
@@
 			)
 		)
-		(property "Footprint" "custom footprints:MP001179"
+		(property "Footprint" "CustomLocalLib:MP001179"
 			(at 215.9 89.916 90)
 			(effects
